File: hardware/the_extender.kicad_sch (KiCad schematic)
At the start: 118 parts, among them J0 TYPE-C 24P QT 143, J1 USB-TYPE-C-010, J2 U231-091N-3BLRC11, J3 PJ-3136-B, J4 PJ-3136-B, J5 AF 10.0 HC6.3, Q1 SSM3J332R,LF, Q2 SSM3J332R,LF, Q3 MMBT3906LT1G, Q4 SSM3J332R,LF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

Commit message: stuff
Parts:
- J0: LCSC Part C388659 -> C5156605
Other:
- note added: "TODO: Ideal Diode, MOSFET, or something"
Changed lines of the file:
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@@
     (stroke (width 0) (type default))
   )
+  (wire (pts (xy 123.19 29.845) (xy 134.62 29.845))
+    (stroke (width 0) (type default))
+  )
   (wire (pts (xy 246.38 227.33) (xy 243.84 227.33))
     (stroke (width 0) (type default))
@@
     (stroke (width 0) (type default))
   )
+  (text "TODO: Ideal Diode, MOSFET, or something" (at 113.03 32.385 0)
+    (effects (font (size 1.27 1.27)) (justify left bottom))
+  )
   (global_label "MIC_T" (shape input) (at 374.65 151.13 0) (fields_autoplaced)
     (effects (font (size 1.27 1.27)) (justify left))
@@
     )
   )
-  (symbol (lib_id "power:+5V") (at 124.46 44.45 0) (unit 1)
+  (symbol (lib_id "power:+5V") (at 123.19 29.845 0) (unit 1)
     (in_bom yes) (on_board yes) (dnp no)
-    (property "Reference" "#PWR0109" (at 124.46 48.26 0)
+    (property "Reference" "#PWR0109" (at 123.19 33.655 0)
       (effects (font (size 1.27 1.27)) hide)
     )
-    (property "Value" "+5V" (at 124.46 40.64 0)
+    (property "Value" "+5V" (at 123.19 24.765 0)
       (effects (font (size 1.27 1.27)))
     )
-    (property "Footprint" "" (at 124.46 44.45 0)
+    (property "Footprint" "" (at 123.19 29.845 0)
       (effects (font (size 1.27 1.27)) hide)
     )
-    (property "Datasheet" "" (at 124.46 44.45 0)
+    (property "Datasheet" "" (at 123.19 29.845 0)
       (effects (font (size 1.27 1.27)) hide)
     )
@@
       (effects (font (size 0 0)) hide)
     )
-    (property "LCSC Part" "C388659" (at 139.7 69.85 0)
+    (property "LCSC Part" "C5156605" (at 139.7 69.85 0)
       (effects (font (size 1.27 1.27)) hide)
     )
@@
     )
   )
+  (symbol (lib_id "power:VBUS") (at 134.62 29.845 0) (unit 1)
+    (in_bom yes) (on_board yes) (dnp no) (fields_autoplaced)
+    (property "Reference" "#PWR064" (at 134.62 33.655 0)
+      (effects (font (size 1.27 1.27)) hide)
+    )
+    (property "Value" "VBUS" (at 134.62 24.765 0)
+      (effects (font (size 1.27 1.27)))
+    )
+    (property "Footprint" "" (at 134.62 29.845 0)
+      (effects (font (size 1.27 1.27)) hide)
+    )
+    (property "Datasheet" "" (at 134.62 29.845 0)
+      (effects (font (size 1.27 1.27)) hide)
+    )
+    (pin "1")
+    (instances
+      (project "the_extender"
+        (path "/e63e39d7-6ac0-4ffd-8aa3-1841a4541b55"
+          (reference "#PWR064") (unit 1)
+        )
+      )
+    )
+  )
   (symbol (lib_id "Device:C") (at 173.99 158.75 0) (mirror y) (unit 1)
     (in_bom yes) (on_board yes) (dnp no)
@@
         )
       )
+    )
+  )
+  (symbol (lib_id "power:VBUS") (at 124.46 44.45 0) (unit 1)
+    (in_bom yes) (on_board yes) (dnp no) (fields_autoplaced)
+    (property "Reference" "#PWR057" (at 124.46 48.26 0)
+      (effects (font (size 1.27 1.27)) hide)
+    )
+    (property "Value" "VBUS" (at 124.46 39.37 0)
+      (effects (font (size 1.27 1.27)))
+    )
+    (property "Footprint" "" (at 124.46 44.45 0)
+      (effects (font (size 1.27 1.27)) hide)
+    )
+    (property "Datasheet" "" (at 124.46 44.45 0)
+      (effects (font (size 1.27 1.27)) hide)
+    )
+    (pin "1")
+    (instances
+      (project "the_extender"
+        (path "/e63e39d7-6ac0-4ffd-8aa3-1841a4541b55"
+          (reference "#PWR057") (unit 1)
+        )
+      )

Commit message: added CC test pads
Parts:
- added TP15: CC2, TestPoint:TestPoint_Pad_D2.0mm, symbol Connector:TestPoint
- added TP16: CC1, TestPoint:TestPoint_Pad_D2.0mm, symbol Connector:TestPoint
Connections:
- net CC1: now also TP16.1
- net CC2: now also TP15.1
Changed lines of the file:
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@@
     )
   )
+  (global_label "CC2" (shape tri_state) (at 314.96 17.78 270) (fields_autoplaced)
+    (effects (font (size 1.27 1.27)) (justify right))
+    (property "Intersheetrefs" "${INTERSHEET_REFS}" (at 314.96 25.626 90)
+      (effects (font (size 1.27 1.27)) (justify right) hide)
+    )
+  )
   (global_label "CC1" (shape bidirectional) (at 119.38 49.53 90) (fields_autoplaced)
     (effects (font (size 1.27 1.27)) (justify left))
@@
     )
   )
+  (global_label "CC1" (shape tri_state) (at 306.705 17.78 270) (fields_autoplaced)
+    (effects (font (size 1.27 1.27)) (justify right))
+    (property "Intersheetrefs" "${INTERSHEET_REFS}" (at 306.705 25.626 90)
+      (effects (font (size 1.27 1.27)) (justify right) hide)
+    )
+  )
   (global_label "SCL" (shape input) (at 213.36 176.53 90) (fields_autoplaced)
     (effects (font (size 1.27 1.27)) (justify left))
@@
     )
   )
+  (symbol (lib_id "Connector:TestPoint") (at 306.705 17.78 0) (unit 1)
+    (in_bom yes) (on_board yes) (dnp no) (fields_autoplaced)
+    (property "Reference" "TP16" (at 308.61 13.208 0)
+      (effects (font (size 1.27 1.27)) (justify left))
+    )
+    (property "Value" "CC1" (at 308.61 15.748 0)
+      (effects (font (size 1.27 1.27)) (justify left))
+    )
+    (property "Footprint" "TestPoint:TestPoint_Pad_D2.0mm" (at 311.785 17.78 0)
+      (effects (font (size 1.27 1.27)) hide)
+    )
+    (property "Datasheet" "~" (at 311.785 17.78 0)
+      (effects (font (size 1.27 1.27)) hide)
+    )
+    (pin "1")
+    (instances
+      (project "the_extender"
+        (path "/e63e39d7-6ac0-4ffd-8aa3-1841a4541b55"
+          (reference "TP16") (unit 1)
+        )
+      )
+    )
+  )
   (symbol (lib_id "power:+3.3VP") (at 212.09 39.37 0) (unit 1)
     (in_bom yes) (on_board yes) (dnp no) (fields_autoplaced)
@@
         )
       )
+    )
+  )
+  (symbol (lib_id "Connector:TestPoint") (at 314.96 17.78 0) (unit 1)
+    (in_bom yes) (on_board yes) (dnp no) (fields_autoplaced)
+    (property "Reference" "TP15" (at 316.865 13.208 0)
+      (effects (font (size 1.27 1.27)) (justify left))
+    )
+    (property "Value" "CC2" (at 316.865 15.748 0)
+      (effects (font (size 1.27 1.27)) (justify left))
+    )
+    (property "Footprint" "TestPoint:TestPoint_Pad_D2.0mm" (at 320.04 17.78 0)
+      (effects (font (size 1.27 1.27)) hide)
+    )
+    (property "Datasheet" "~" (at 320.04 17.78 0)
+      (effects (font (size 1.27 1.27)) hide)
+    )
+    (pin "1")
+    (instances
+      (project "the_extender"
+        (path "/e63e39d7-6ac0-4ffd-8aa3-1841a4541b55"
+          (reference "TP15") (unit 1)
+        )
+      )

Commit message: idk
Parts:
- TP15, TP16: footprint TestPoint:TestPoint_Pad_D2.0mm -> TestPoint:TestPoint_Pad_D1.0mm
Changed lines of the file:
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@@
       (effects (font (size 1.27 1.27)) (justify left))
     )
-    (property "Footprint" "TestPoint:TestPoint_Pad_D2.0mm" (at 311.785 17.78 0)
+    (property "Footprint" "TestPoint:TestPoint_Pad_D1.0mm" (at 311.785 17.78 0)
       (effects (font (size 1.27 1.27)) hide)
     )
@@
       (effects (font (size 1.27 1.27)) (justify left))
     )
-    (property "Footprint" "TestPoint:TestPoint_Pad_D2.0mm" (at 320.04 17.78 0)
-      (effects (font (size 1.27 1.27)) hide)
-    )
+    (property "Footprint" "TestPoint:TestPoint_Pad_D1.0mm" (at 320.04 17.78 0)
+      (effects (font (size 1.27 1.27)) hide)
+    )

Commit message: debug TX pad
Parts:
- added TP17: RX, TestPoint:TestPoint_Pad_D1.0mm, symbol Connector:TestPoint
- added TP18: TX, TestPoint:TestPoint_Pad_D1.0mm, symbol Connector:TestPoint
Connections:
- net UART_RX: now reaches U2.27 (GPIO16)
- net UART_RX: now also TP17.1
- net UART_TX: now reaches U2.28 (GPIO17)
- net UART_TX: now also TP18.1
- no-connect marks 56 -> 54
Changed lines of the file:
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@@
   )
   (no_connect (at 374.65 90.17))
-  (no_connect (at 374.65 115.57))
   (no_connect (at 240.03 100.33))
   (no_connect (at 240.03 97.79))
@@
   (no_connect (at 50.8 137.16))
   (no_connect (at 80.01 163.83))
-  (no_connect (at 374.65 118.11))
   (no_connect (at 374.65 92.71))
   (no_connect (at 39.37 161.29))
@@
     )
   )
+  (global_label "UART_RX" (shape output) (at 298.45 31.75 270) (fields_autoplaced)
+    (effects (font (size 1.27 1.27)) (justify right))
+    (property "Intersheetrefs" "${INTERSHEET_REFS}" (at 298.45 42.839 90)
+      (effects (font (size 1.27 1.27)) (justify right) hide)
+    )
+  )
   (global_label "SCL" (shape output) (at 374.65 100.33 0) (fields_autoplaced)
     (effects (font (size 1.27 1.27)) (justify left))
@@
     )
   )
+  (global_label "UART_TX" (shape output) (at 374.65 118.11 0) (fields_autoplaced)
+    (effects (font (size 1.27 1.27)) (justify left))
+    (property "Intersheetrefs" "${INTERSHEET_REFS}" (at 385.4366 118.11 0)
+      (effects (font (size 1.27 1.27)) (justify left) hide)
+    )
+  )
   (global_label "CC_USB_INT" (shape input) (at 374.65 110.49 0) (fields_autoplaced)
     (effects (font (size 1.27 1.27)) (justify left))
@@
     )
   )
+  (global_label "UART_TX" (shape input) (at 285.75 31.75 270) (fields_autoplaced)
+    (effects (font (size 1.27 1.27)) (justify right))
+    (property "Intersheetrefs" "${INTERSHEET_REFS}" (at 285.75 42.5366 90)
+      (effects (font (size 1.27 1.27)) (justify right) hide)
+    )
+  )
   (global_label "SND_EEPROM_CS" (shape input) (at 374.65 128.27 0) (fields_autoplaced)
     (effects (font (size 1.27 1.27)) (justify left))
@@
     )
   )
+  (global_label "UART_RX" (shape input) (at 374.65 115.57 0) (fields_autoplaced)
+    (effects (font (size 1.27 1.27)) (justify left))
+    (property "Intersheetrefs" "${INTERSHEET_REFS}" (at 385.739 115.57 0)
+      (effects (font (size 1.27 1.27)) (justify left) hide)
+    )
+  )
   (global_label "MIC_R" (shape bidirectional) (at 43.18 267.97 0) (fields_autoplaced)
     (effects (font (size 1.27 1.27)) (justify left))
@@
     )
   )
+  (symbol (lib_id "Connector:TestPoint") (at 285.75 31.75 0) (unit 1)
+    (in_bom yes) (on_board yes) (dnp no) (fields_autoplaced)
+    (property "Reference" "TP18" (at 288.29 27.178 0)
+      (effects (font (size 1.27 1.27)) (justify left))
+    )
+    (property "Value" "TX" (at 288.29 29.718 0)
+      (effects (font (size 1.27 1.27)) (justify left))
+    )
+    (property "Footprint" "TestPoint:TestPoint_Pad_D1.0mm" (at 290.83 31.75 0)
+      (effects (font (size 1.27 1.27)) hide)
+    )
+    (property "Datasheet" "~" (at 290.83 31.75 0)
+      (effects (font (size 1.27 1.27)) hide)
+    )
+    (pin "1")
+    (instances
+      (project "the_extender"
+        (path "/e63e39d7-6ac0-4ffd-8aa3-1841a4541b55"
+          (reference "TP18") (unit 1)
+        )
+      )
+    )
+  )
   (symbol (lib_id "Device:C") (at 363.22 53.34 90) (unit 1)
     (in_bom yes) (on_board yes) (dnp no)
@@
         )
       )
+    )
+  )
+  (symbol (lib_id "Connector:TestPoint") (at 298.45 31.75 0) (unit 1)
+    (in_bom no) (on_board no) (dnp yes) (fields_autoplaced)
+    (property "Reference" "TP17" (at 300.99 27.178 0)
+      (effects (font (size 1.27 1.27)) (justify left))
+    )
+    (property "Value" "RX" (at 300.99 29.718 0)
+      (effects (font (size 1.27 1.27)) (justify left))
+    )
+    (property "Footprint" "TestPoint:TestPoint_Pad_D1.0mm" (at 303.53 31.75 0)
+      (effects (font (size 1.27 1.27)) hide)
+    )
+    (property "Datasheet" "~" (at 303.53 31.75 0)
+      (effects (font (size 1.27 1.27)) hide)
+    )
+    (pin "1")
+    (instances
+      (project "the_extender"
+        (path "/e63e39d7-6ac0-4ffd-8aa3-1841a4541b55"
+          (reference "TP17") (unit 1)
+        )
+      )

Commit message: todo
Other:
- note added: "TODO: WTF does this do???"
- note added: "TODO: limit voltage to 3V6"
- company: (none) -> H3
- title: (none) -> The Extender
Changed lines of the file:
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@@
 (kicad_sch (version 20230121) (generator eeschema)
   (paper "A3")
+  (title_block
+    (title "The Extender")
+    (rev "v0.0")
+    (company "H3")
+  )
   (junction (at 247.65 180.34) (diameter 0) (color 0 0 0 0)
   )
@@
     (stroke (width 0) (type default))
   )
+  (rectangle (start 153.67 241.3) (end 213.995 281.305)
+    (stroke (width 0) (type default))
+    (fill (type none))
+  )
+  (text "TODO: WTF does this do???\n" (at 167.005 240.665 0)
+    (effects (font (size 1.27 1.27)) (justify left bottom))
+  )
   (text "TODO: Ideal Diode, MOSFET, or something" (at 113.03 32.385 0)
     (effects (font (size 1.27 1.27)) (justify left bottom))
   )
+  (text "TODO: limit voltage to 3V6" (at 401.32 127 90)
+    (effects (font (size 1.27 1.27)) (justify left bottom))
+  )

Commit message: now i know
Other:
- note added: "Oh, this is Overvoltage Protection"
- note removed: "TODO: WTF does this do???"
Changed lines of the file:
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@@
   (junction (at 243.84 248.92) (diameter 0) (color 0 0 0 0)
   )
+  (junction (at 162.56 248.92) (diameter 0) (color 0 0 0 0)
+  )
   (junction (at 210.82 180.34) (diameter 0) (color 0 0 0 0)
   )
@@
   )
   (junction (at 231.14 227.33) (diameter 0) (color 0 0 0 0)
-  )
-  (junction (at 158.75 256.54) (diameter 0) (color 0 0 0 0)
   )
   (no_connect (at 374.65 90.17))
@@
     (stroke (width 0) (type default))
   )
+  (wire (pts (xy 166.37 256.54) (xy 162.56 256.54))
+    (stroke (width 0) (type default))
+  )
   (wire (pts (xy 77.47 133.35) (xy 81.28 133.35))
     (stroke (width 0) (type default))
@@
     (stroke (width 0) (type default))
   )
+  (wire (pts (xy 162.56 256.54) (xy 162.56 248.92))
+    (stroke (width 0) (type default))
+  )
   (wire (pts (xy 327.66 57.15) (xy 330.2 57.15))
     (stroke (width 0) (type default))
@@
     (stroke (width 0) (type default))
   )
-  (wire (pts (xy 158.75 248.92) (xy 180.34 248.92))
+  (wire (pts (xy 158.75 248.92) (xy 162.56 248.92))
     (stroke (width 0) (type default))
   )
@@
     (stroke (width 0) (type default))
   )
-  (wire (pts (xy 158.75 256.54) (xy 166.37 256.54))
-    (stroke (width 0) (type default))
-  )
   (wire (pts (xy 158.75 248.92) (xy 158.75 256.54))
     (stroke (width 0) (type default))
@@
     (stroke (width 0) (type default))
   )
+  (wire (pts (xy 162.56 248.92) (xy 180.34 248.92))
+    (stroke (width 0) (type default))
+  )
   (wire (pts (xy 297.18 67.31) (xy 297.18 69.85))
     (stroke (width 0) (type default))
@@
     (fill (type none))
   )
-  (text "TODO: WTF does this do???\n" (at 167.005 240.665 0)
+  (text "Oh, this is Overvoltage Protection" (at 167.005 240.665 0)
     (effects (font (size 1.27 1.27)) (justify left bottom))
   )

Commit message: todo
Other:
- note added: "Maybe remove OVP and replace with discharge mosfet, audio reset, etc"
- note removed: "Oh, this is Overvoltage Protection"
Changed lines of the file:
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@@
     (stroke (width 0) (type default))
   )
-  (rectangle (start 153.67 241.3) (end 213.995 281.305)
+  (rectangle (start 156.21 240.665) (end 213.995 281.305)
     (stroke (width 0) (type default))
     (fill (type none))
-  )
-  (text "Oh, this is Overvoltage Protection" (at 167.005 240.665 0)
-    (effects (font (size 1.27 1.27)) (justify left bottom))
   )
   (text "TODO: Ideal Diode, MOSFET, or something" (at 113.03 32.385 0)
@@
     (effects (font (size 1.27 1.27)) (justify left bottom))
   )
+  (text "Maybe remove OVP and replace with discharge mosfet, audio reset, etc"
+    (at 144.145 240.03 0)
+    (effects (font (size 1.27 1.27)) (justify left bottom))
+  )

Commit message: giving up on eeprom emulation, not enough board space
Parts:
- R10: value 2k -> 2k2
- R13: value 1k -> 4k7
- R9: value 2k -> 1k
- TP17: now fitted; now in the parts list
- TP18: footprint TestPoint:TestPoint_Pad_D1.0mm -> TestPoint:TestPoint_Pad_D2.0mm
- TP3, TP6, TP8: footprint TestPoint:TestPoint_Pad_D2.0mm -> TestPoint:TestPoint_Pad_D1.0mm
Connections:
- net +3V3: now also C44.1, R18.1, R20.1, U4.12 (VCONN), U4.13 (VCONN), U4.3 (VDD), U4.4 (VDD)
- net +BATT: no longer C44.1, R18.1, R20.1, U4.12 (VCONN), U4.13 (VCONN), U4.3 (VDD), U4.4 (VDD)
- net CLK_24M: now also U2.29 (GPIO18); no longer U2.2 (GPIO0)
- net SND_EEPROM_CS: no longer U2.32 (GPIO21)
- net SND_EEPROM_DR: no longer U2.29 (GPIO18)
- net SND_EEPROM_DW: no longer U2.30 (GPIO19)
- net SND_EEPROM_SCK: no longer U2.31 (GPIO20)
- net SND_LED_O: now also R13.2; no longer R10.2
- net at R9.1: now also D2.4 (RA); no longer D2.3 (BA)
- net at R13.1: now also D2.3 (BA); no longer D2.4 (RA)
- net RP_LED_R: now reaches U2.9 (GPIO7)
- net RP_LED_R: now also R9.2
- net MCU_LED renamed RP_LED_G
- net RP_LED_G: now also R10.2; no longer R9.2
- net SND_LED_R: no longer names the net of U6.19 (LEDR)
- net SND_LED_R: no longer R13.2
- no-connect marks 54 -> 58
Other:
- note added: "TODO: limit voltage to 3V6 Resistor arrays maybe... or Zeners... so little space!"
- note added: "TODO: make 5VA switchable"
- note removed: "TODO: limit voltage to 3V6"
