File: cable/usb_c_ffc/usb_c_ffc.kicad_sch (KiCad schematic)
At the start: 7 parts, among them J1 Conn_01x15_Socket, J2 Conn_01x15_Socket, J3 Conn_01x15_Socket, J4 Conn_01x15_Socket, J5 Conn_01x15_Socket, P1 TC-003LS, P2 TC-003LS

Commit message: cable pcb panel
Other:
- note added: "FlatFlexCable: JS10A-15P-050-4-8"
Changed lines of the file:
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@@
     (fill (type none))
+  )
+  (text "FlatFlexCable: JS10A-15P-050-4-8" (at 139.065 113.665 0)
+    (effects (font (size 1.27 1.27)) (justify left bottom))
   )
   (text "Layout: VBUS VBUS VBUS GND CC GND D- D+ GND RX- RX+ GND TX- TX+ GND GND"
