File: cable/USB2/usb_c_2.kicad_pcb (KiCad board)
At the start: 2 copper layers, 11.5 x 11.5 mm, 2 parts, among them J1 Conn_02x03_Odd_Even, P1 TC-003LS

Commit message: change routing
Routing:
- net /CC: track 7.48 -> 13.8 mm, vias 1 -> 0
- net VBUS: track 8.21 -> 9.91 mm, vias 3 -> 4
Changed lines of the file:
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@@
   )
   (segment (start 53.25 49) (end 53.75 49.5) (width 0.25) (layer "F.Cu") (net 2))
+  (segment (start 50.75 49) (end 50.25 49.5) (width 0.25) (layer "F.Cu") (net 2))
   (segment (start 50.75 46.09) (end 50.75 44.75) (width 0.25) (layer "F.Cu") (net 2))
   (segment (start 53.25 46.09) (end 53.25 48) (width 0.25) (layer "F.Cu") (net 2))
@@
   (segment (start 53.25 46.09) (end 53.25 44.75) (width 0.25) (layer "F.Cu") (net 2))
   (segment (start 50.75 46.09) (end 50.75 48) (width 0.25) (layer "F.Cu") (net 2))
+  (segment (start 50.75 48) (end 50.75 49) (width 0.25) (layer "F.Cu") (net 2))
   (via (at 53.25 44.75) (size 0.8) (drill 0.4) (layers "F.Cu" "B.Cu") (net 2))
   (via (at 50.75 44.75) (size 0.8) (drill 0.4) (layers "F.Cu" "B.Cu") (net 2))
+  (via (at 50.25 49.5) (size 0.8) (drill 0.4) (layers "F.Cu" "B.Cu") (net 2))
   (via (at 53.75 49.5) (size 0.8) (drill 0.4) (layers "F.Cu" "B.Cu") (net 2))
-  (segment (start 53.25 52.75) (end 53.25 50.25) (width 0.2) (layer "F.Cu") (net 3))
-  (segment (start 52.25 49.25) (end 52.25 48) (width 0.2) (layer "F.Cu") (net 3))
-  (segment (start 53.25 50.25) (end 52.25 49.25) (width 0.2) (layer "F.Cu") (net 3))
   (segment (start 54.54 54.04) (end 53.25 52.75) (width 0.2) (layer "F.Cu") (net 3))
-  (segment (start 50.77 49.5) (end 50.25 49.5) (width 0.25) (layer "F.Cu") (net 4))
-  (segment (start 51.25 48) (end 51.25 49.02) (width 0.25) (layer "F.Cu") (net 4))
-  (segment (start 51.25 49.02) (end 50.77 49.5) (width 0.25) (layer "F.Cu") (net 4))
-  (via (at 50.25 49.5) (size 0.8) (drill 0.4) (layers "F.Cu" "B.Cu") (net 4))
-  (segment (start 50.825 50.075) (end 50.825 52.865) (width 0.25) (layer "B.Cu") (net 4))
-  (segment (start 50.25 49.5) (end 50.825 50.075) (width 0.25) (layer "B.Cu") (net 4))
-  (segment (start 50.825 52.865) (end 52 54.04) (width 0.25) (layer "B.Cu") (net 4))
-  (segment (start 50.75 52.75) (end 50.75 50.25) (width 0.2) (layer "F.Cu") (net 6))
-  (segment (start 51.75 49.25) (end 51.75 48) (width 0.2) (layer "F.Cu") (net 6))
-  (segment (start 50.75 50.25) (end 51.75 49.25) (width 0.2) (layer "F.Cu") (net 6))
+  (segment (start 52.25 49.65) (end 52.25 48) (width 0.2) (layer "F.Cu") (net 3))
+  (segment (start 53.25 52.75) (end 53.25 50.65) (width 0.2) (layer "F.Cu") (net 3))
+  (segment (start 53.25 50.65) (end 52.25 49.65) (width 0.2) (layer "F.Cu") (net 3))
+  (segment (start 48.499695 50.225) (end 48.1 50.624695) (width 0.2) (layer "F.Cu") (net 4))
+  (segment (start 50.550305 50.225) (end 48.499695 50.225) (width 0.2) (layer "F.Cu") (net 4))
+  (segment (start 50.715 55.325) (end 52 54.04) (width 0.2) (layer "F.Cu") (net 4))
+  (segment (start 48.825 55.325) (end 50.715 55.325) (width 0.2) (layer "F.Cu") (net 4))
+  (segment (start 48.1 50.624695) (end 48.1 54.44223) (width 0.2) (layer "F.Cu") (net 4))
+  (segment (start 51.25 49.525305) (end 50.550305 50.225) (width 0.2) (layer "F.Cu") (net 4))
+  (segment (start 48.1 54.44223) (end 48.15522 54.65522) (width 0.2) (layer "F.Cu") (net 4))
+  (segment (start 48.15522 54.65522) (end 48.825 55.325) (width 0.2) (layer "F.Cu") (net 4))
+  (segment (start 51.25 48) (end 51.25 49.525305) (width 0.2) (layer "F.Cu") (net 4))
   (segment (start 49.46 54.04) (end 50.75 52.75) (width 0.2) (layer "F.Cu") (net 6))
+  (segment (start 50.75 50.65) (end 51.75 49.65) (width 0.2) (layer "F.Cu") (net 6))
+  (segment (start 51.75 49.65) (end 51.75 48) (width 0.2) (layer "F.Cu") (net 6))
+  (segment (start 50.75 52.75) (end 50.75 50.65) (width 0.2) (layer "F.Cu") (net 6))
   (zone (net 1) (net_name "GND") (layers "F&B.Cu") (hatch edge 0.5)
     (connect_pads yes (clearance 0.2))
@@
     (polygon
       (pts
-        (xy 51 52.5)
+        (xy 50.8 50.2)
+        (xy 50.8 52.5)
         (xy 53.25 52.5)
         (xy 53.25 50.25)
-        (xy 54.25 49.85)
+        (xy 54.25 49.9)
         (xy 54.25 49.1)
-        (xy 53.75 48.75)
+        (xy 53.75 48.8)
         (xy 53.75 44.25)
         (xy 50.25 44.25)
-        (xy 50.25 48.5)
-        (xy 51 49.5)
+        (xy 50.2 48.8)
+        (xy 49.8 49.1)
+        (xy 49.8 49.9)
       )
     )
